File: ADXL372_Board/ADXL372_circuit.brd (EAGLE design)
At the start: 45 x 45 mm, 53 parts, among them CN1 FH12-08S-1SH, IC1 STM32L051C6, IC2 ADXL345BCCZ, IC3 ADXL372BCCZ-RL7, IC4 SI7006-A20-IM, IC6 MX25R1635FM1IL0, IC7 74AHC1G14DCK, IC8 LP5907MFX-2.5/NOPB, Q2 BSS138W, SW1 DHT-4235A, SW2 B3U-1000P-2P-SMD, SW3 JS202011SCQN, Y1 16MHZ_X053201602002, Y2 3.2768KHZ

Commit message: Update board design
Parts:
- removed Q2: BSS138W, BSS138W:SOT323-R
- added TR2: BSS138W, BSS138W:SOT323-R
- C24: value 10uf -> 100nf; device OPL_Capacitor:C0805 -> OPL_Capacitor:C0603
- moved SW1 43.9 mm to (36.2, 4.31), turned to 0 degrees
- moved R6 38.5 mm to (6.35, 24.1), turned to 270 degrees
- moved SW2 36.9 mm to (7.87, 21.1), turned to 180 degrees
- moved C23 36.3 mm to (6.35, 26.7), turned to 180 degrees
- moved IC7 32.0 mm to (8.64, 26.4)
- moved C22 30.2 mm to (41.1, 24.6), turned to 180 degrees
- moved C16 30.2 mm to (3.81, 14.4)
- moved C25 28.8 mm to (30.2, 30.5), turned to 270 degrees
- moved C24 26.8 mm to (30.2, 32.5), turned to 270 degrees
- moved R1 20.6 mm to (6.10, 8.76), turned to 90 degrees
- moved TP8 14.1 mm to (18.3, 7.87), flipped to the bottom
- moved C17 11.5 mm to (8.76, 39.9), turned to 90 degrees
- moved TP7 11.1 mm to (20.8, 9.40), flipped to the bottom
- moved C5 10.1 mm to (40.0, 12.6), turned to 0 degrees
- moved TP5 7.71 mm to (25.9, 9.14), flipped to the bottom
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Connections:
- net N$3 renamed RESET
- removed net I2C2_SCL: IC4.6, R2.1
- removed net I2C2_SDA: IC4.1, R3.1
- removed net VCC: C24.2, C25.2, IC8.5
- net +2V5: now also C16.2, C17.2, C23.2, C24.2, C25.2, C4.2, C5.2, IC2.1, IC2.6, IC4.5, IC6.8, IC7.5, IC8.5, R1.2, R2.2, R3.2, R6.2
- net +3V3: no longer C16.2, C17.2, C23.2, C4.2, C5.2, IC2.1, IC2.6, IC4.5, IC6.8, IC7.5, R1.2, R2.2, R3.2, R6.2
- net GND: now also TR2.2; no longer Q2.2
- net I2C1_SCL: now also IC4.6, R2.1
- net I2C1_SDA: now also IC4.1, R3.1
- net N$19: now also TR2.3; no longer Q2.3
- net N$4: now also TR2.1; no longer Q2.1
Routing:
- net +2V5: track 24.7 -> 60.8 mm
- net SPI2_MISO: track 34.2 -> 0.00 mm, vias 2 -> 0
- net GND: track 20.0 -> 50.2 mm
- net FLASH_MEMORY: track 28.9 -> 0.02 mm, vias 2 -> 0
- net I2C1_SCL: track 0.00 -> 27.5 mm, vias 0 -> 2
- net SPI2_SCK: track 26.3 -> 0.00 mm, vias 2 -> 0
- net I2C1_SDA: track 0.00 -> 24.6 mm, vias 0 -> 2
- net +BAT: track 0.00 -> 21.8 mm, vias 0 -> 1
- net SPI2_MOSI: track 20.9 -> 0.00 mm, vias 2 -> 0
- net RESET: track 0.00 -> 20.8 mm
- net ADXL372_CS: track 0.00 -> 19.4 mm, vias 0 -> 2
- net SPI1_MOSI: track 16.8 -> 32.0 mm
- net SPI1_MISO: track 18.7 -> 31.9 mm, vias 0 -> 2
- net +3V3: track 9.83 -> 22.5 mm
- net 372_INT2: track 11.9 -> 0.00 mm, vias 2 -> 0
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