File: ADXL372_Board/ADXL372_circuit.brd (EAGLE design)
At the start: 45 x 45 mm, 53 parts, among them CN1 FH12-08S-1SH, IC1 STM32L051C6, IC2 ADXL345BCCZ, IC3 ADXL372BCCZ-RL7, IC4 SI7006-A20-IM, IC6 MX25R1635FM1IL0, IC7 74AHC1G14DCK, IC8 LP5907MFX-2.5/NOPB, SW1 DHT-4235A, SW2 B3U-1000P-2P-SMD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

Commit message: Update board design
Parts:
- moved TP4 37.8 mm to (12.3, 41.9)
- moved TP6 36.9 mm to (9.98, 42.0)
- moved TP8 34.6 mm to (31.4, 39.9)
- moved TP5 34.4 mm to (11.3, 40.3)
- moved TP7 33.4 mm to (8.38, 40.4)
- moved TP3 30.1 mm to (33.4, 38.9)
- moved C22 2.29 mm to (42.4, 26.5)
- moved C14 2.25 mm to (39.9, 26.8)
- moved C17 1.98 mm to (10.0, 38.4)
- moved IC6 1.98 mm to (10.2, 34.5)
Routing:
- net +2V5: track 60.8 -> 182.3 mm, vias 0 -> 5
- net MODE_LED: track 0.00 -> 45.7 mm, vias 0 -> 2
- net N$9: track 0.00 -> 35.2 mm, vias 0 -> 1
- net N$10: track 0.00 -> 32.2 mm, vias 0 -> 1
- net N$8: track 0.00 -> 32.2 mm, vias 0 -> 1
- net FLASH_MEMORY: track 0.02 -> 30.8 mm, vias 0 -> 2
- net SPI2_MISO: track 0.00 -> 28.1 mm, vias 0 -> 2
- net N$6: track 0.00 -> 27.6 mm, vias 0 -> 1
- net 372_INT1: track 0.00 -> 25.9 mm, vias 0 -> 2
- net N$7: track 0.00 -> 24.9 mm, vias 0 -> 1
- net 372_INT2: track 0.00 -> 21.3 mm, vias 0 -> 2
- net SPI2_SCK: track 0.00 -> 19.2 mm, vias 0 -> 2
- net SPI2_MOSI: track 0.00 -> 18.6 mm, vias 0 -> 2
- net N$11: track 0.00 -> 17.8 mm, vias 0 -> 1
- net GND: track 50.2 -> 64.9 mm, vias 0 -> 1
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- added copper zone on layer 1, net GND
- added copper zone on layer 16, net GND

Commit message: Update board design
Parts:
- added C15: 100nf, OPL_Capacitor:C0603
- added C7: 10uf, OPL_Capacitor:C0805
- added R7, R8: 10K 1/10W, OPL_Resistor:R0603
- C10, C9: value 8pf -> 10pf
- TP5, TP6, TP7: value TPB1,27 -> TPSB1,27
- X1: value 16MHZ_X053201602002 -> 8MHz
- moved TP8 30.2 mm to (31.9, 9.63)
- moved Y2 1.93 mm to (25.9, 13.9)
- moved C20 1.93 mm to (25.0, 11.2)
- moved C21 1.93 mm to (27.2, 11.2)
- moved TP1 1.52 mm to (16.5, 28.7)
- moved C24 1.28 mm to (31.5, 32.7)
- moved C25 1.28 mm to (31.5, 30.6)
- moved C22 0.90 mm to (41.8, 25.9)
- moved C14 0.82 mm to (39.8, 26.0)
- moved C8 0.76 mm to (17.9, 30.4)
- renumbered Y1 to X1
Connections:
- removed net N$10: IC1.43, TP7.TP
- removed net N$11: IC1.21, TP8.TP
- removed net N$8: IC1.41, TP5.TP
- removed net N$9: IC1.42, TP6.TP
- new net I2C1_SMBA: IC1.41
- new net N$12: IC1.44, R7.1, R8.1
- new net TP5: IC1.45, TP5.TP
- new net TP6: IC1.46, TP6.TP
- new net TP7: IC1.21, TP7.TP
- net +2V5: now also C15.2, C7.2, IC1.24, R8.2
- net GND: now also C15.1, C7.1, IC1.8, R7.2
- net I2C1_SCL: now also IC1.42; no longer IC1.45
- net I2C1_SDA: now also IC1.43; no longer IC1.46
- net RESET: now also TP8.TP
Routing:
- net GND: track 64.9 -> 359.4 mm, vias 1 -> 136
- net +2V5: track 182.3 -> 245.9 mm, vias 5 -> 8
- net TP7: track 0.00 -> 41.5 mm, vias 0 -> 3
- net TP5: track 0.00 -> 39.1 mm, vias 0 -> 1
- net N$12: track 0.00 -> 38.6 mm, vias 0 -> 2
- net N$9: track 35.2 -> 0.00 mm, vias 1 -> 0
- net TP6: track 0.00 -> 34.8 mm, vias 0 -> 1
- net N$10: track 32.2 -> 0.00 mm, vias 1 -> 0
- net N$8: track 32.2 -> 0.00 mm, vias 1 -> 0
- net N$11: track 17.8 -> 0.00 mm, vias 1 -> 0
- net SPI1_MISO: track 31.9 -> 41.1 mm
- net ADXL345_CS: track 25.0 -> 32.7 mm
- net MODE_LED: track 45.7 -> 52.5 mm
- net FLASH_MEMORY: track 30.8 -> 37.1 mm
- net RESET: track 20.8 -> 26.9 mm, vias 0 -> 1
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
Commit message: Update Board design
Change CN1
Parts:
- CN1: value FH12-08S-1SH -> 505568-0871; device con-hirose:FH12-08S-1SH -> 505568-0871:MOLEX_505568-0871
- moved CN1 1.94 mm to (22.4, 40.0), turned to 0 degrees
- renumbered Y2 to X2
Connections:
- net +3V3: now also CN1.8; no longer CN1.1
- net GND: now also CN1.1, CN1.2, CN1.S1, CN1.S2; no longer CN1.7, CN1.8
- net USART1_CK: now also CN1.7; no longer CN1.2
- net USART1_CTS: now also CN1.4; no longer CN1.5
- net USART1_RTS: now also CN1.3; no longer CN1.6
- net USART1_RX: now also CN1.5; no longer CN1.4
- net USART1_TX: now also CN1.6; no longer CN1.3
Routing:
- net GND: track 359.4 -> 348.4 mm, vias 136 -> 131
- net +2V5: track 245.9 -> 241.1 mm
- net USART1_CK: track 11.2 -> 12.8 mm
- net USART1_RTS: track 10.5 -> 12.1 mm
- net USART1_TX: track 11.0 -> 12.5 mm
- net USART1_RX: track 10.8 -> 12.2 mm
- net USART1_CTS: track 10.6 -> 11.9 mm
- net +3V3: track 18.7 -> 19.4 mm

Commit message: Update Board design
Routing:
- net GND: track 348.4 -> 351.7 mm, vias 131 -> 134
Changed lines of the file:
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@@
 <wire x1="9.2924" y1="25.5541" x2="9.286" y2="25.566" width="0.1524" layer="1"/>
 <wire x1="11.6155" y1="22.8736" x2="11.632709375" y2="22.827684375" width="0.1524" layer="1"/>
-<wire x1="19.1209" y1="37.5742" x2="19.1209" y2="38.5992" width="0.1524" layer="1"/>
 <wire x1="17.6913" y1="36.1446" x2="19.1209" y2="37.5742" width="0.1524" layer="1"/>
 <wire x1="17.6913" y1="32.3447" x2="17.6913" y2="36.1446" width="0.1524" layer="1"/>
 <wire x1="17.6913" y1="32.3447" x2="17.526" y2="32.258" width="0.1524" layer="1"/>
-<wire x1="16.132" y1="39.6714" x2="17.0763" y2="38.7271" width="0.1524" layer="1"/>
+<wire x1="16.132" y1="39.6714" x2="17.0684" y2="38.735" width="0.1524" layer="1"/>
+<wire x1="17.0684" y1="38.735" x2="17.0763" y2="38.7271" width="0.1524" layer="1"/>
 <wire x1="10.5433" y1="39.6714" x2="16.132" y2="39.6714" width="0.1524" layer="1"/>
 <wire x1="9.2924" y1="38.4205" x2="10.5433" y2="39.6714" width="0.1524" layer="1"/>
 <wire x1="9.2924" y1="38.4205" x2="9.271" y2="38.354" width="0.1524" layer="1"/>
-<wire x1="28.4133" y1="34.4383" x2="28.4133" y2="32.578653125" width="0.1524" layer="1"/>
+<wire x1="28.4133" y1="34.2383" x2="28.4133" y2="32.578653125" width="0.1524" layer="1"/>
 <wire x1="28.4133" y1="32.578653125" x2="28.4133" y2="32.166" width="0.1524" layer="1"/>
-<wire x1="25.2282" y1="37.6234" x2="28.4133" y2="34.4383" width="0.1524" layer="1"/>
+<wire x1="26.3258" y1="36.3258" x2="28.4133" y2="34.2383" width="0.1524" layer="1"/>
 <wire x1="28.4133" y1="32.166" x2="28.448" y2="32.0548" width="0.1524" layer="1"/>
 <via x="20.3718" y="29.3068" extent="1-16" drill="0.3"/>
@@
 <vertex x="26.2636" y="27.9908"/>
 </polygon>
+<wire x1="19.1209" y1="38.9209" x2="19.3" y2="39.1" width="0.1524" layer="1"/>
+<wire x1="19.3" y1="39.1" x2="19.3" y2="39.9574" width="0.1524" layer="1"/>
+<wire x1="19.3" y1="39.9574" x2="19.2778" y2="39.9796" width="0.1524" layer="1"/>
+<wire x1="19.1209" y1="37.5742" x2="19.1209" y2="38.4" width="0.1524" layer="1"/>
+<wire x1="19.1209" y1="38.4" x2="19.1209" y2="38.9209" width="0.1524" layer="1"/>
+<wire x1="18.0278" y1="38.9278" x2="18.0278" y2="39.9796" width="0.1524" layer="1"/>
+<wire x1="17.145" y1="38.735" x2="17.0684" y2="38.735" width="0.1524" layer="1"/>
+<wire x1="17.145" y1="38.735" x2="17.835" y2="38.735" width="0.1524" layer="1"/>
+<wire x1="18.0278" y1="38.9278" x2="17.835" y2="38.735" width="0.1524" layer="1"/>
+<wire x1="17.835" y1="38.735" x2="18.17" y2="38.4" width="0.1524" layer="1"/>
+<wire x1="18.17" y1="38.4" x2="19.1209" y2="38.4" width="0.1524" layer="1"/>
+<via x="25.6" y="37.5" extent="1-16" drill="0.3"/>
+<via x="18.7" y="42.1" extent="1-16" drill="0.3"/>
+<via x="26" y="42.1" extent="1-16" drill="0.3"/>
 </signal>
 <signal name="N$1">
@@
 <wire x1="18.2836" y1="20.0706" x2="18.543465625" y2="19.916734375" width="0.1524" layer="1"/>
 </signal>
-<signal name="N$3">
-<via x="25.6" y="37.5" extent="1-16" drill="0.3"/>
-</signal>
-<signal name="N$8">
-<via x="18.7" y="42.1" extent="1-16" drill="0.3"/>
-</signal>
-<signal name="N$9">
-<via x="26" y="42.1" extent="1-16" drill="0.3"/>
-</signal>
 </signals>
