File: ADXL372_Board/ADXL372_circuit.brd (EAGLE design)
At the start: 45 x 45 mm, 57 parts, among them CN1 505568-0871, IC1 STM32L051C6, IC2 ADXL345BCCZ, IC3 ADXL372BCCZ-RL7, IC4 SI7006-A20-IM, IC6 MX25R1635FM1IL0, IC7 74AHC1G14DCK, IC8 LP5907MFX-2.5/NOPB, SW1 DHT-4235A, SW2 B3U-1000P-2P-SMD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

Commit message: Update
Parts:
- C20, C21: value 12.5pf -> 7pf
- SW1: value DHT-4235A -> PTS645SK50SMTR92LFS; device OPL_Switch:SW4-SMD-4.2X3.2X2.5MM -> PTS645SK50SMTR92LFS:SW_PTS645SK50SMTR92LFS
- X2: value 3.2768KHZ -> 32.768KHZ
- moved C13 3.28 mm to (32.1, 10.8)
- moved TP8 2.85 mm to (29.5, 11.2)
- moved SW1 2.51 mm to (34.7, 6.30)
- moved R7 2.00 mm to (27.3, 4.95)
- moved R8 2.00 mm to (24.9, 4.95)
Routing:
- net RESET: track 26.9 -> 18.5 mm
- net GND: track 351.7 -> 343.8 mm, vias 134 -> 127
- net +2V5: track 241.1 -> 239.2 mm
- net N$12: track 38.6 -> 37.3 mm

Commit message: Correction battery pattern
Routing:
- net GND: vias 127 -> 128
Changed lines of the file:
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@@
 <setting verticaltext="up"/>
 </settings>
-<grid distance="25" unitdist="mil" unit="mil" style="dots" multiple="1" display="yes" altdistance="5" altunitdist="mil" altunit="mil"/>
+<grid distance="5" unitdist="mil" unit="mil" style="dots" multiple="1" display="yes" altdistance="5" altunitdist="mil" altunit="mil"/>
 <layers>
 <layer number="1" name="Top" color="4" fill="1" visible="yes" active="yes"/>
@@
 <layer number="25" name="tNames" color="7" fill="1" visible="yes" active="yes"/>
 <layer number="26" name="bNames" color="7" fill="1" visible="yes" active="yes"/>
-<layer number="27" name="tValues" color="7" fill="1" visible="yes" active="yes"/>
-<layer number="28" name="bValues" color="7" fill="1" visible="yes" active="yes"/>
+<layer number="27" name="tValues" color="7" fill="1" visible="no" active="yes"/>
+<layer number="28" name="bValues" color="7" fill="1" visible="no" active="yes"/>
 <layer number="29" name="tStop" color="7" fill="3" visible="no" active="yes"/>
 <layer number="30" name="bStop" color="7" fill="6" visible="no" active="yes"/>
@@
 <element name="C24" library="OPL_Capacitor" package="C0603" package3d_urn="urn:adsk.eagle:package:8004287/1" value="100nf" x="31.496" y="32.6644" smashed="yes" rot="R270">
 <attribute name="MPN" value="CC0603KRX7R9BB104" x="36.322" y="37.2364" size="1.778" layer="27" rot="R270" display="off"/>
+<attribute name="NAME" x="32.766" y="32.9184" size="0.635" layer="33" ratio="10" rot="R180"/>
 <attribute name="NAME" x="27.7368" y="32.2326" size="0.889" layer="25" ratio="11"/>
-<attribute name="NAME" x="32.766" y="32.9184" size="0.635" layer="33" ratio="10" rot="R180"/>
 <attribute name="VALUE" x="32.766" y="34.2519" size="0.635" layer="27" ratio="10" rot="R180"/>
 </element>
@@
 <element name="C15" library="OPL_Capacitor" package="C0603" package3d_urn="urn:adsk.eagle:package:8004287/1" value="100nf" x="27.5082" y="28.3972" smashed="yes" rot="R270">
 <attribute name="MPN" value="CC0603KRX7R9BB104" x="27.5082" y="28.3972" size="1.778" layer="27" rot="R270" display="off"/>
+<attribute name="NAME" x="27.7114" y="26.5938" size="0.8128" layer="25" ratio="10"/>
 <attribute name="NAME" x="28.7782" y="28.6512" size="0.635" layer="33" ratio="10" rot="R180"/>
-<attribute name="NAME" x="27.7114" y="26.5938" size="0.8128" layer="25" ratio="10"/>
 <attribute name="VALUE" x="28.7782" y="29.9847" size="0.635" layer="27" ratio="10" rot="R180"/>
 </element>
@@
 <wire x1="32.893" y1="10.795" x2="35.179" y2="8.509" width="0.254" layer="1"/>
 <wire x1="35.179" y1="8.509" x2="35.179" y2="4.05" width="0.254" layer="1"/>
+<polygon width="0.1524" layer="16" pour="cutout">
+<vertex x="25.781" y="26.416"/>
+<vertex x="22.86" y="26.416"/>
+<vertex x="22.86" y="20.828"/>
+<vertex x="22.987" y="20.701"/>
+<vertex x="24.384" y="20.701"/>
+<vertex x="24.384" y="19.177"/>
+<vertex x="24.511" y="19.05"/>
+<vertex x="26.797" y="19.05"/>
+<vertex x="26.797" y="19.812"/>
+<vertex x="29.21" y="19.812"/>
+<vertex x="29.337" y="19.939"/>
+<vertex x="29.337" y="26.162"/>
+<vertex x="29.21" y="26.289"/>
+<vertex x="29.083" y="26.416"/>
+</polygon>
+<via x="21.844" y="25.527" extent="1-16" drill="0.35"/>
 </signal>
 <signal name="N$1">
