File: ADXL372_Board/ADXL372_circuit.sch (EAGLE design)
At the start: 53 parts, among them CN1 FH12-08S-1SH, IC1 STM32L051C6, IC2 ADXL345BCCZ, IC3 ADXL372BCCZ-RL7, IC4 SI7006-A20-IM, IC6 MX25R1635FM1IL0, IC7 74AHC1G14DCK, IC8 LP5907MFX-2.5/NOPB, SW1 DHT-4235A, SW2 B3U-1000P-2P-SMD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

Commit message: Update board design
Parts:
- added C15: 100nf, OPL_Capacitor:CERAMIC-100NF-50V-10%-X7R(0603)
- added C7: 10uf, OPL_Capacitor:CERAMIC-10UF-10V-(-20%～+80%)-Y5V(0805)
- added R7, R8: 10K 1/10W, OPL_Resistor:SMD-RES-10K-5%-1/10W(0603)
- C10, C9: value 8pf -> 10pf
- TP5, TP6, TP7: value TPB1,27 -> TPSB1,27; device testpad:TPB1,27 -> testpad:TPSB1,27
- X1: value 16MHZ_X053201602002 -> 8MHz
- renumbered Y1 to X1
Connections:
- removed net N$10: IC1.PB7, TP7.TP
- removed net N$11: IC1.PB10, TP8.TP
- removed net N$8: IC1.PB5, TP5.TP
- removed net N$9: IC1.PB6, TP6.TP
- new net I2C1_SMBA: IC1.PB5
- new net N$12: IC1.BOOT0, R7.1, R8.1
- new net TP5: IC1.PB8, TP5.PP
- new net TP6: IC1.PB9, TP6.PP
- new net TP7: IC1.PB10, TP7.PP
- net +2V5: now also C15.2, C7.2, IC1.VDDIO2, R8.2
- net GND: now also C15.1, C7.1, IC1.VSSA, R7.2
- net I2C1_SCL: now also IC1.PB6; no longer IC1.PB8
- net I2C1_SDA: now also IC1.PB7; no longer IC1.PB9
- net RESET: now also TP8.TP
Other:
- moved on the sheet: C13, SW1, TP8

Commit message: Update Board design
Change CN1
Parts:
- CN1: value FH12-08S-1SH -> 505568-0871; device con-hirose:FH12-08S-1SH -> 505568-0871:505568-0871
- renumbered Y2 to X2
Connections:
- net +3V3: now also CN1.8; no longer CN1-1.1
- net GND: now also CN1.1, CN1.2, CN1.SHIELD; no longer CN1-7.1, CN1-8.1
- net USART1_CK: now also CN1.7; no longer CN1-2.1
- net USART1_CTS: now also CN1.4; no longer CN1-5.1
- net USART1_RTS: now also CN1.3; no longer CN1-6.1
- net USART1_RX: now also CN1.5; no longer CN1-4.1
- net USART1_TX: now also CN1.6; no longer CN1-3.1

Commit message: Update
Parts:
- C20, C21: value 12.5pf -> 7pf
- SW1: value DHT-4235A -> PTS645SK50SMTR92LFS; device OPL_Switch:SMD-BUTTON-TOP-DHT-4235A(4P-4.2X3.2MM) -> PTS645SK50SMTR92LFS:PTS645SK50SMTR92LFS
- X2: value 3.2768KHZ -> 32.768KHZ
Connections:
- net GND: now also SW1.3, SW1.4; no longer SW1.B0, SW1.B1
- net RESET: now also SW1.1; no longer SW1.A0
Changed lines of the file:
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@@
 <setting verticaltext="up"/>
 </settings>
-<grid distance="0.1" unitdist="inch" unit="inch" style="lines" multiple="1" display="no" altdistance="0.01" altunitdist="inch" altunit="inch"/>
+<grid distance="0.05" unitdist="inch" unit="inch" style="dots" multiple="1" display="yes" altdistance="0.01" altunitdist="inch" altunit="inch"/>
 <layers>
 <layer number="1" name="Top" color="4" fill="1" visible="no" active="no"/>
@@
 <part name="C10" library="OPL_Capacitor" library_urn="urn:adsk.eagle:library:8004261" deviceset="CERAMIC-10PF-50V-5%-NPO(0603)" device="" package3d_urn="urn:adsk.eagle:package:8004287/1" value="10pf"/>
 <part name="C13" library="OPL_Capacitor" deviceset="CERAMIC-100NF-50V-10%-X7R(0603)" device="" package3d_urn="urn:adsk.eagle:package:8004287/1" value="100nf"/>
-<part name="SW1" library="OPL_Switch" deviceset="SMD-BUTTON-TOP-DHT-4235A(4P-4.2X3.2MM)" device="" package3d_urn="urn:adsk.eagle:package:8005116/1" value="DHT-4235A"/>
 <part name="SUPPLY11" library="supply2" library_urn="urn:adsk.eagle:library:372" deviceset="GND" device=""/>
 <part name="SUPPLY12" library="supply2" library_urn="urn:adsk.eagle:library:372" deviceset="GND" device=""/>
@@
 <part name="C18" library="OPL_Capacitor" deviceset="CERAMIC-100NF-50V-10%-X7R(0603)" device="" package3d_urn="urn:adsk.eagle:package:8004287/1" value="100nf"/>
 <part name="C19" library="OPL_Capacitor" deviceset="CERAMIC-10UF-10V-(-20%～+80%)-Y5V(0805)" device="" package3d_urn="urn:adsk.eagle:package:8004286/1" value="10uf"/>
-<part name="X2" library="OPL_Crystal Oscillator" library_urn="urn:adsk.eagle:library:8004402" deviceset="SMD-CRYSTAL-32.768KHZ-12.5PF-20PPM-90K(2P-L2.0X1.2MM)" device="" package3d_urn="urn:adsk.eagle:package:8004453/1" value="3.2768KHZ"/>
-<part name="C20" library="OPL_Capacitor" deviceset="CERAMIC-10PF-50V-5%-NPO(0603)" device="" package3d_urn="urn:adsk.eagle:package:8004287/1" value="12.5pf"/>
-<part name="C21" library="OPL_Capacitor" deviceset="CERAMIC-10PF-50V-5%-NPO(0603)" device="" package3d_urn="urn:adsk.eagle:package:8004287/1" value="12.5pf"/>
+<part name="X2" library="OPL_Crystal Oscillator" library_urn="urn:adsk.eagle:library:8004402" deviceset="SMD-CRYSTAL-32.768KHZ-12.5PF-20PPM-90K(2P-L2.0X1.2MM)" device="" package3d_urn="urn:adsk.eagle:package:8004453/1" value="32.768KHZ"/>
+<part name="C20" library="OPL_Capacitor" deviceset="CERAMIC-10PF-50V-5%-NPO(0603)" device="" package3d_urn="urn:adsk.eagle:package:8004287/1" value="7pf"/>
+<part name="C21" library="OPL_Capacitor" deviceset="CERAMIC-10PF-50V-5%-NPO(0603)" device="" package3d_urn="urn:adsk.eagle:package:8004287/1" value="7pf"/>
 <part name="SUPPLY22" library="supply2" library_urn="urn:adsk.eagle:library:372" deviceset="GND" device=""/>
 <part name="VCC10" library="supply1" library_urn="urn:adsk.eagle:library:371" deviceset="+3V3" device="" value="+2V5"/>
@@
 <part name="VCC2" library="supply1" library_urn="urn:adsk.eagle:library:371" deviceset="+3V3" device="" value="+2V5"/>
 <part name="SUPPLY24" library="supply2" library_urn="urn:adsk.eagle:library:372" deviceset="GND" device=""/>
-<part name="IC7" library="74xx-little-us" library_urn="urn:adsk.eagle:library:87" deviceset="74*1G14" device="DCK" package3d_urn="urn:adsk.eagle:package:2405/1" technology="AHC"/>
+<part name="IC7" library="74xx-little-us" library_urn="urn:adsk.eagle:library:87" deviceset="74*1G14" device="DCK" package3d_urn="urn:adsk.eagle:package:2405/2" technology="AHC"/>
 <part name="C23" library="OPL_Capacitor" deviceset="CERAMIC-100NF-50V-10%-X7R(0603)" device="" package3d_urn="urn:adsk.eagle:package:8004287/1" value="100nf"/>
 <part name="VCC11" library="supply1" library_urn="urn:adsk.eagle:library:371" deviceset="+3V3" device="" value="+2V5"/>
@@
 <part name="CN1" library="505568-0871" library_urn="urn:adsk.eagle:library:14702135" deviceset="505568-0871" device="" package3d_urn="urn:adsk.eagle:package:14702138/1" override_package3d_urn="urn:adsk.eagle:package:14702165/2" override_package_urn="urn:adsk.eagle:footprint:14702136/1"/>
 <part name="SUPPLY15" library="supply2" library_urn="urn:adsk.eagle:library:372" deviceset="GND" device=""/>
+<part name="SW1" library="PTS645SK50SMTR92LFS" library_urn="urn:adsk.eagle:library:14741174" deviceset="PTS645SK50SMTR92LFS" device="" package3d_urn="urn:adsk.eagle:package:14741177/2"/>
 </parts>
 <sheets>
@@
 <attribute name="VALUE" x="251.46" y="167.64" size="1.27" layer="96" ratio="10" rot="R90"/>
 </instance>
-<instance part="SW1" gate="G$1" x="269.24" y="175.26" smashed="yes">
-<attribute name="NAME" x="264.16" y="180.34" size="1.27" layer="95" ratio="10"/>
-<attribute name="VALUE" x="264.16" y="168.91" size="1.27" layer="96" ratio="10"/>
-</instance>
 <instance part="SUPPLY11" gate="GND" x="248.92" y="162.56" smashed="yes">
 <attribute name="VALUE" x="247.015" y="159.385" size="1.778" layer="96"/>
@@
 </instance>
 <instance part="TP5" gate="G$1" x="241.3" y="144.78" smashed="yes" rot="R270">
-<attribute name="NAME" x="242.57" y="146.05" size="1.778" layer="95" rot="R270"/>
+<attribute name="NAME" x="242.57" y="143.764" size="1.778" layer="95"/>
 <attribute name="TP_SIGNAL_NAME" x="240.03" y="143.51" size="1.778" layer="97" rot="R270"/>
 </instance>
 <instance part="TP6" gate="G$1" x="241.3" y="142.24" smashed="yes" rot="R270">
-<attribute name="NAME" x="246.38" y="142.875" size="1.778" layer="95" rot="R180"/>
+<attribute name="NAME" x="242.57" y="141.224" size="1.778" layer="95"/>
 <attribute name="TP_SIGNAL_NAME" x="240.03" y="140.97" size="1.778" layer="97" rot="R270"/>
 </instance>
 <instance part="TP7" gate="G$1" x="241.3" y="139.7" smashed="yes" rot="R270">
-<attribute name="NAME" x="246.38" y="140.335" size="1.778" layer="95" rot="R180"/>
+<attribute name="NAME" x="242.57" y="138.684" size="1.778" layer="95"/>
 <attribute name="TP_SIGNAL_NAME" x="240.03" y="138.43" size="1.778" layer="97" rot="R270"/>
 </instance>
@@
 <instance part="SUPPLY15" gate="GND" x="114.3" y="147.32" smashed="yes">
 <attribute name="VALUE" x="112.395" y="144.145" size="1.778" layer="96"/>
+</instance>
+<instance part="SW1" gate="G$1" x="269.24" y="175.26" smashed="yes">
+<attribute name="NAME" x="264.662759375" y="184.6644" size="1.780040625" layer="95"/>
+<attribute name="VALUE" x="264.15211875" y="181.85258125" size="1.780759375" layer="96"/>
 </instance>
 </instances>
@@
 </segment>
 <segment>
-<pinref part="SW1" gate="G$1" pin="B1"/>
-<wire x1="278.13" y1="172.72" x2="280.67" y2="172.72" width="0.1524" layer="91"/>
+<wire x1="276.86" y1="172.72" x2="280.67" y2="172.72" width="0.1524" layer="91"/>
 <pinref part="SUPPLY12" gate="GND" pin="GND"/>
 <wire x1="280.67" y1="172.72" x2="280.67" y2="166.37" width="0.1524" layer="91"/>
-<pinref part="SW1" gate="G$1" pin="B0"/>
 <wire x1="280.67" y1="166.37" x2="280.67" y2="163.83" width="0.1524" layer="91"/>
-<wire x1="260.35" y1="172.72" x2="257.81" y2="172.72" width="0.1524" layer="91"/>
+<wire x1="261.62" y1="172.72" x2="257.81" y2="172.72" width="0.1524" layer="91"/>
 <wire x1="257.81" y1="172.72" x2="257.81" y2="166.37" width="0.1524" layer="91"/>
 <wire x1="257.81" y1="166.37" x2="280.67" y2="166.37" width="0.1524" layer="91"/>
 <junction x="280.67" y="166.37"/>
+<pinref part="SW1" gate="G$1" pin="3"/>
+<pinref part="SW1" gate="G$1" pin="4"/>
 </segment>
 <segment>
@@
 <net name="RESET" class="0">
 <segment>
-<pinref part="SW1" gate="G$1" pin="A0"/>
 <wire x1="220.98" y1="177.8" x2="248.92" y2="177.8" width="0.1524" layer="91"/>
 <pinref part="C13" gate="G$1" pin="2"/>
-<wire x1="248.92" y1="177.8" x2="260.35" y2="177.8" width="0.1524" layer="91"/>
+<wire x1="248.92" y1="177.8" x2="261.62" y2="177.8" width="0.1524" layer="91"/>
 <wire x1="248.92" y1="175.26" x2="248.92" y2="177.8" width="0.1524" layer="91"/>
 <junction x="248.92" y="177.8"/>
@@
 <junction x="220.98" y="177.8"/>
 <pinref part="TP8" gate="G$1" pin="TP"/>
+<pinref part="SW1" gate="G$1" pin="1"/>
 </segment>
 </net>
